File: atmega8/pcb/led_pixel/led_pixel.kicad_pcb (KiCad board)
At the start: 2 copper layers, 50 x 50 mm, 61 parts, among them CON101 10PIN_ISP_AVR, IC1 ATMEGA8-AI, P1 USB_OTG, P3 CONN_01X03, P4 CONN_01X03, P5 CONN_01X04, SW1 SW_DIP_x08, U1 MC78M05CDT, U2 PT4115, U3 PT4115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

Commit message: generated documentation and gerber files
Other:
- board text added: "04/2017"
Changed lines of the file:
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@@
-(kicad_pcb (version 20170123) (host pcbnew "(2017-04-15 revision 60310b3d3)-makepkg")
+(kicad_pcb (version 20160815) (host pcbnew "(2017-01-09 revision c2fb336)-makepkg")
   (general
     (links 152)
     (no_connects 0)
-    (area 123.588999 62.6392 180.289286 118.28372)
+    (area 124.924999 64.924999 175.075001 115.075001)
     (thickness 1.6)
-    (drawings 4)
+    (drawings 5)
     (tracks 1033)
     (zones 0)
@@
   )
   (setup
-    (last_trace_width 0.5)
+    (last_trace_width 0.3)
     (user_trace_width 0.3)
     (user_trace_width 0.5)
@@
       (layerselection 0x010fc_ffffffff)
       (usegerberextensions true)
-      (excludeedgelayer true)
+      (excludeedgelayer false)
       (linewidth 0.100000)
       (plotframeref true)
@@
       (psa4output false)
       (plotreference true)
-      (plotvalue true)
+      (plotvalue false)
       (plotinvisibletext false)
       (padsonsilk false)
-      (subtractmaskfromsilk true)
+      (subtractmaskfromsilk false)
       (outputformat 4)
       (mirror false)
       (drillshape 2)
       (scaleselection 1)
-      (outputdirectory doku))
+      (outputdirectory doc))
   )
   (net 0 "")
@@
     (add_net VCC)
   )
+  (module proz_led:LED_SMD_RGB_3W (layer F.Cu)
+    (at 150 90)
+    (fp_text reference D6 (at -6.5532 3.4036) (layer F.SilkS)
+      (effects (font (size 1 1) (thickness 0.15)))
+    )
+    (fp_text value LED_RGB (at 0 -4.8) (layer F.Fab)
+      (effects (font (size 1 1) (thickness 0.15)))
+    )
+    (fp_circle (center 0 0) (end 4 0) (layer F.SilkS) (width 0.15))
+    (pad "" smd circle (at 0 0) (size 9 9) (layers B.Mask))
+    (pad "" smd circle (at 0 0) (size 7.5 7.5) (layers F.Mask))
+    (pad 1 smd rect (at 6.5 -1.8) (size 3 1) (layers F.Cu F.Paste F.Mask)
+      (net 9 /LED_R_K))
+    (pad 2 smd rect (at 6.5 0) (size 3 1) (layers F.Cu F.Paste F.Mask)
+      (net 8 /LED_G_K))
+    (pad 3 smd rect (at 6.5 1.8) (size 3 1) (layers F.Cu F.Paste F.Mask)
+      (net 7 /LED_B_K))
+    (pad 4 smd rect (at -6.5 1.8) (size 3 1) (layers F.Cu F.Paste F.Mask)
+      (net 6 /LED_B_A))
+    (pad 5 smd rect (at -6.5 0) (size 3 1) (layers F.Cu F.Paste F.Mask)
+      (net 5 /LED_G_A))
+    (pad 6 smd rect (at -6.5 -1.8) (size 3 1) (layers F.Cu F.Paste F.Mask)
+      (net 4 /LED_R_A))
+  )
   (module Crystals:Crystal_SMD_HC49-SD_HandSoldering (layer F.Cu)
     (at 153.75 67.75 180)
@@
       (net 25 "Net-(D4-Pad2)"))
   )
-  (module proz_led:LED_SMD_RGB_3W (layer F.Cu)
-    (at 150 90)
-    (fp_text reference D6 (at -4.191 3.683) (layer F.SilkS)
-      (effects (font (size 1 1) (thickness 0.15)))
-    )
-    (fp_text value LED_RGB (at 0 -4.8) (layer F.Fab)
-      (effects (font (size 1 1) (thickness 0.15)))
-    )
-    (fp_circle (center 0 0) (end 4 0) (layer F.SilkS) (width 0.15))
-    (pad "" smd circle (at 0 0) (size 7.5 7.5) (layers F.Mask))
-    (pad 1 smd rect (at 6.5 -1.8) (size 3 1) (layers F.Cu F.Paste F.Mask)
-      (net 9 /LED_R_K))
-    (pad 2 smd rect (at 6.5 0) (size 3 1) (layers F.Cu F.Paste F.Mask)
-      (net 8 /LED_G_K))
-    (pad 3 smd rect (at 6.5 1.8) (size 3 1) (layers F.Cu F.Paste F.Mask)
-      (net 7 /LED_B_K))
-    (pad 4 smd rect (at -6.5 1.8) (size 3 1) (layers F.Cu F.Paste F.Mask)
-      (net 6 /LED_B_A))
-    (pad 5 smd rect (at -6.5 0) (size 3 1) (layers F.Cu F.Paste F.Mask)
-      (net 5 /LED_G_A))
-    (pad 6 smd rect (at -6.5 -1.8) (size 3 1) (layers F.Cu F.Paste F.Mask)
-      (net 4 /LED_R_A))
-  )
   (module Mounting_Holes:MountingHole_3.2mm_M3_DIN965 (layer F.Cu)
     (at 138.5 86)
@@
     (tags "capacitor 0603")
     (attr smd)
-    (fp_text reference C3 (at 0 -1.524 180) (layer F.SilkS)
+    (fp_text reference C3 (at -2.8448 0 180) (layer F.SilkS)
       (effects (font (size 1 1) (thickness 0.15)))
     )
@@
     (tags "capacitor 0603")
     (attr smd)
-    (fp_text reference C5 (at 0 -1.9) (layer F.SilkS)
+    (fp_text reference C5 (at 0 -1.3208) (layer F.SilkS)
       (effects (font (size 1 1) (thickness 0.15)))
     )
@@
     (tags "resistor 0603")
     (attr smd)
-    (fp_text reference R1 (at 1.143 -1.524 180) (layer F.SilkS)
+    (fp_text reference R1 (at 0.5842 -1.4224 180) (layer F.SilkS)
       (effects (font (size 1 1) (thickness 0.15)))
     )
@@
     )
   )
+  (gr_text 04/2017 (at 156.4516 67.9528) (layer B.Cu)
+    (effects (font (size 1.5 1.5) (thickness 0.3)) (justify mirror))
+  )
   (gr_line (start 175 65) (end 125 65) (layer Edge.Cuts) (width 0.15))

Commit message: added pcb number and revision
re generated all docu and gerber data
- ordered this one as rev 1.0
Other:
- board text added: "05/2017 Rev: 1.0 0003"
- board text removed: "04/2017"
Changed lines of the file:
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@@
-(kicad_pcb (version 20170123) (host pcbnew "(2017-05-08 revision d4e41c4f9)-makepkg")
+(kicad_pcb (version 20170123) (host pcbnew "(2017-05-12 revision b823d0b78)-makepkg")
   (general
     (links 152)
@@
   (title_block
     (title led_pixel_atmega8)
-    (date 2017-05-10)
+    (date 2017-05-13)
     (rev 1.0)
     (company shimatta)
@@
       (layerselection 0x010fc_ffffffff)
       (usegerberextensions true)
-      (excludeedgelayer true)
+      (excludeedgelayer false)
       (linewidth 0.100000)
-      (plotframeref false)
+      (plotframeref true)
       (viasonmask false)
       (mode 1)
@@
       (psa4output false)
       (plotreference true)
-      (plotvalue false)
+      (plotvalue true)
       (plotinvisibletext false)
       (padsonsilk false)
       (subtractmaskfromsilk false)
-      (outputformat 1)
+      (outputformat 4)
       (mirror false)
       (drillshape 0)
       (scaleselection 1)
-      (outputdirectory gerber))
+      (outputdirectory doc))
   )
   (net 0 "")
@@
     )
   )
-  (gr_text 04/2017 (at 156.4516 67.9528) (layer B.Cu)
-    (effects (font (size 1.5 1.5) (thickness 0.3)) (justify mirror))
+  (gr_text "05/2017\nRev: 1.0\n0003" (at 155.715 68.6005) (layer B.Cu)
+    (effects (font (size 0.8 0.8) (thickness 0.2)) (justify mirror))
   )
   (gr_line (start 175 65) (end 125 65) (layer Edge.Cuts) (width 0.15))
