File: stm32f030/pcb/led_pixel_stm32f030/led_pixel_stm32f030.sch (KiCad schematic (older format))
At the start: 18 parts

Commit message: designed a first draft of the backplane of the dynamic adressing LED Pixels
started with pcb design of the STM32 version
Parts:
- removed D?: SS310, Diodes_SMD:D_SMA_Standard, symbol D_Schottky
- removed P?: CONN_01X04, Socket_Strips:Socket_Strip_Straight_1x04, symbol CONN_01X04
- added C1, C2: 100n, Capacitors_SMD:C_0603_HandSoldering, symbol C
- added Q1: BC107, TO_SOT_Packages_SMD:SOT-23, symbol Q_NPN_BEC
- added R1, R3, R5: 10k, Resistors_SMD:R_0603_HandSoldering, symbol R
- added R2: 220, Resistors_SMD:R_0603_HandSoldering, symbol R
- added R4: 1k, Resistors_SMD:R_0603_HandSoldering, symbol R
- C3, C4: renamed from C?; value C -> 20p; footprint (none) -> Capacitors_SMD:C_0603_HandSoldering
- C6, C7: renamed from C?; footprint Capacitors_SMD:C_0805_HandSoldering -> Capacitors_SMD:C_0603_HandSoldering
- CON1: renamed from CON?; footprint (none) -> proz_connectors:TC2050-IDC
- R6: renamed from R?; value R -> 6k8; footprint (none) -> Resistors_SMD:R_0603_HandSoldering
- R8: renamed from R?; value R -> 10k; footprint (none) -> Resistors_SMD:R_0603_HandSoldering
- U3: renamed from U?; footprint (none) -> TO_SOT_Packages_SMD:SOT-223
- gave numbers to parts that had none: 8
Connections:
- net #RS485_RE is gone; now on net RS485_DE: U2.2 (RE)
- net #RESET: now also Q1.3 (C), R3.1
- net +3V3: now also C1.1, C2.1, R3.2
- net GND: now also CON1.3 (GND), C1.2, C2.2, Q1.2 (E), R1.1, R5.1
- net PWM_LED_B: now also U1.18 (I2C1_SDA/TIM17_BKIN/TIM1_CH3/USART1_RX/PA10)
- net PWM_LED_G: now also U1.17 (I2C1_SCL/TIM1_CH2/USART1_TX/PA9)
- net PWM_LED_R: now also U1.10 (ADC_IN4/SPI1_NSS/TIM14_CH1/USART1_CK/PA4)
- net PWM_LED_W: now also U1.14 (PB1/ADC_IN9/TIM14_CH1/TIM1_CH3N/TIM3_CH4)
- net RS485_DE: now also U1.7 (ADC_IN1/USART1_DE/USART1_RTS/PA1)
- net RS485_RX: now also CON1.9 (TX/nTRST), U1.9 (ADC_IN3/USART1_RX/PA3)
- net RS485_TX: now also CON1.7 (RX/RTCLK), U1.8 (ADC_IN2/USART1_TX/PA2)
- net SWDIO: now reaches CON1.2 (TMS/SWDIO)
- net SWDIO: now also U1.19 (IR_OUT/SYS_SWDIO/PA13)
- net SWCLK: now reaches CON1.4 (TCK/SWCLK)
- net SWCLK: now also U1.20 (SYS_SWCLK/USART1_TX/PA14)
- net TESTMODE: now reaches CON1.5 (GND/Supply/Testmode)
- net TESTMODE: now also U1.6 (ADC_IN0/RTC_TAMP2/SYS_WKUP1/USART1_CTS/PA0)
- net at U1.1 (BOOT0): now also R1.2
- net SPI_CLK: now reaches U1.11 (ADC_IN5/SPI1_SCK/PA5)
- net SPI_MISO: now reaches U1.12 (ADC_IN6/SPI1_MISO/TIM16_CH1/TIM1_BKIN/TIM3_CH1/PA6)
- net SPI_MOSI: now reaches U1.13 (ADC_IN7/SPI1_MOSI/TIM14_CH1/TIM17_CH1/TIM1_CH1N/TIM3_CH2/PA7)
- net at C4.1, Y1.2: now also R2.1; no longer U1.3 (PF1/RCC_OSC_OUT)
- net RS485_B renamed RS485_N
- net RS485_a renamed RS485_P
- new net: R2.2, U1.3 (PF1/RCC_OSC_OUT)
- new net: Q1.1 (B), R4.1, R5.2
- new net RESET_IN: R4.2
- no-connect marks 0 -> 2
Other:
- moved on the sheet: C3, C4, CON1, U1, Y1

Commit message: made a first layout draft...
well okay, wouldn´t call it layout yet ;)

- next step make it look like a Layout XD
Connections:
- net PWM_LED_B: now also U1.14 (PB1/ADC_IN9/TIM14_CH1/TIM1_CH3N/TIM3_CH4); no longer U1.18 (I2C1_SDA/TIM17_BKIN/TIM1_CH3/USART1_RX/PA10)
- net PWM_LED_W: now also U1.18 (I2C1_SDA/TIM17_BKIN/TIM1_CH3/USART1_RX/PA10); no longer U1.14 (PB1/ADC_IN9/TIM14_CH1/TIM1_CH3N/TIM3_CH4)
Changed lines of the file:
@@
 $EndComp
 $Comp
-L GND #PWR22
+L GND #PWR01
 U 1 1 58FD042C
 P 850 7300
-F 0 "#PWR22" H 850 7050 50  0001 C CNN
+F 0 "#PWR01" H 850 7050 50  0001 C CNN
 F 1 "GND" H 855 7127 50  0000 C CNN
 F 2 "" H 850 7300 50  0000 C CNN
@@
 $EndComp
 $Comp
-L GND #PWR23
+L GND #PWR02
 U 1 1 58FD042D
 P 1200 7300
-F 0 "#PWR23" H 1200 7050 50  0001 C CNN
+F 0 "#PWR02" H 1200 7050 50  0001 C CNN
 F 1 "GND" H 1205 7127 50  0000 C CNN
 F 2 "" H 1200 7300 50  0000 C CNN
@@
 $EndComp
 $Comp
-L GND #PWR24
+L GND #PWR03
 U 1 1 58FD042E
 P 1850 7300
-F 0 "#PWR24" H 1850 7050 50  0001 C CNN
+F 0 "#PWR03" H 1850 7050 50  0001 C CNN
 F 1 "GND" H 1855 7127 50  0000 C CNN
 F 2 "" H 1850 7300 50  0000 C CNN
@@
 $EndComp
 $Comp
-L GND #PWR25
+L GND #PWR04
 U 1 1 58FD042F
 P 2500 7300
-F 0 "#PWR25" H 2500 7050 50  0001 C CNN
+F 0 "#PWR04" H 2500 7050 50  0001 C CNN
 F 1 "GND" H 2505 7127 50  0000 C CNN
 F 2 "" H 2500 7300 50  0000 C CNN
@@
 $EndComp
 $Comp
-L GND #PWR26
+L GND #PWR05
 U 1 1 58FD0430
 P 2900 7300
-F 0 "#PWR26" H 2900 7050 50  0001 C CNN
+F 0 "#PWR05" H 2900 7050 50  0001 C CNN
 F 1 "GND" H 2905 7127 50  0000 C CNN
 F 2 "" H 2900 7300 50  0000 C CNN
@@
 RS485_DE
 $Comp
-L +5V #PWR16
+L +5V #PWR06
 U 1 1 58FD044C
 P 10350 5400
-F 0 "#PWR16" H 10350 5250 50  0001 C CNN
+F 0 "#PWR06" H 10350 5250 50  0001 C CNN
 F 1 "+5V" H 10365 5573 50  0000 C CNN
 F 2 "" H 10350 5400 50  0000 C CNN
@@
 $EndComp
 $Comp
-L GND #PWR19
+L GND #PWR07
 U 1 1 58FD044D
 P 10350 6000
-F 0 "#PWR19" H 10350 5750 50  0001 C CNN
+F 0 "#PWR07" H 10350 5750 50  0001 C CNN
 F 1 "GND" H 10355 5827 50  0000 C CNN
 F 2 "" H 10350 6000 50  0000 C CNN
@@
 $EndComp
 $Comp
-L +5V #PWR15
+L +5V #PWR08
 U 1 1 58FD0472
 P 7900 5400
-F 0 "#PWR15" H 7900 5250 50  0001 C CNN
+F 0 "#PWR08" H 7900 5250 50  0001 C CNN
 F 1 "+5V" H 7915 5573 50  0000 C CNN
 F 2 "" H 7900 5400 50  0000 C CNN
@@
 $EndComp
 $Comp
-L GND #PWR17
+L GND #PWR09
 U 1 1 58FD0473
 P 7900 6000
-F 0 "#PWR17" H 7900 5750 50  0001 C CNN
+F 0 "#PWR09" H 7900 5750 50  0001 C CNN
 F 1 "GND" H 7905 5827 50  0000 C CNN
 F 2 "" H 7900 6000 50  0000 C CNN
@@
 $EndComp
 $Comp
-L GND #PWR10
+L GND #PWR010
 U 1 1 58FDD5A4
 P 3100 3850
-F 0 "#PWR10" H 3100 3600 50  0001 C CNN
+F 0 "#PWR010" H 3100 3600 50  0001 C CNN
 F 1 "GND" H 3105 3677 50  0000 C CNN
 F 2 "" H 3100 3850 50  0001 C CNN
@@
 $EndComp
 $Comp
-L GND #PWR11
+L GND #PWR011
 U 1 1 58FDE385
 P 5450 3850
-F 0 "#PWR11" H 5450 3600 50  0001 C CNN
+F 0 "#PWR011" H 5450 3600 50  0001 C CNN
 F 1 "GND" H 5455 3677 50  0000 C CNN
 F 2 "" H 5450 3850 50  0001 C CNN
@@
 $EndComp
 $Comp
-L +3V3 #PWR21
+L +3V3 #PWR012
 U 1 1 58FDEE90
 P 2900 6400
-F 0 "#PWR21" H 2900 6250 50  0001 C CNN
+F 0 "#PWR012" H 2900 6250 50  0001 C CNN
 F 1 "+3V3" H 2915 6573 50  0000 C CNN
 F 2 "" H 2900 6400 50  0001 C CNN
@@
 $EndComp
 $Comp
-L +3V3 #PWR1
+L +3V3 #PWR013
 U 1 1 58FDEFD6
 P 5450 850
-F 0 "#PWR1" H 5450 700 50  0001 C CNN
+F 0 "#PWR013" H 5450 700 50  0001 C CNN
 F 1 "+3V3" H 5465 1023 50  0000 C CNN
 F 2 "" H 5450 850 50  0001 C CNN
@@
 $EndComp
 $Comp
-L +5V #PWR20
+L +5V #PWR014
 U 1 1 58FDF76E
 P 850 6400
-F 0 "#PWR20" H 850 6250 50  0001 C CNN
+F 0 "#PWR014" H 850 6250 50  0001 C CNN
 F 1 "+5V" H 865 6573 50  0000 C CNN
 F 2 "" H 850 6400 50  0000 C CNN
@@
 $EndComp
 $Comp
-L +3V3 #PWR3
+L +3V3 #PWR015
 U 1 1 58FE057D
 P 1900 1000
-F 0 "#PWR3" H 1900 850 50  0001 C CNN
+F 0 "#PWR015" H 1900 850 50  0001 C CNN
 F 1 "+3V3" H 1915 1173 50  0000 C CNN
 F 2 "" H 1900 1000 50  0001 C CNN
@@
 Text Label 7250 2600 0    60   ~ 0
 PWM_LED_G
+Text Label 3800 3650 0    60   ~ 0
+PWM_LED_B
 Text Label 7250 2700 0    60   ~ 0
-PWM_LED_B
-Text Label 3800 3650 0    60   ~ 0
 PWM_LED_W
 Text Label 10750 5650 0    60   ~ 0
@@
 $EndComp
 $Comp
-L GND #PWR18
+L GND #PWR016
 U 1 1 58FE56F9
 P 8550 6000
-F 0 "#PWR18" H 8550 5750 50  0001 C CNN
+F 0 "#PWR016" H 8550 5750 50  0001 C CNN
 F 1 "GND" H 8555 5827 50  0000 C CNN
 F 2 "" H 8550 6000 50  0000 C CNN
@@
 RS485_N
 $Comp
-L VCC #PWR5
+L VCC #PWR017
 U 1 1 5906753A
 P 9750 1150
-F 0 "#PWR5" H 9750 1000 50  0001 C CNN
+F 0 "#PWR017" H 9750 1000 50  0001 C CNN
 F 1 "VCC" H 9800 1350 50  0000 C CNN
 F 2 "" H 9750 1150 50  0001 C CNN
@@
 $EndComp
 $Comp
-L GND #PWR8
+L GND #PWR018
 U 1 1 59068160
 P 9750 3200
-F 0 "#PWR8" H 9750 2950 50  0001 C CNN
+F 0 "#PWR018" H 9750 2950 50  0001 C CNN
 F 1 "GND" H 9755 3027 50  0000 C CNN
 F 2 "" H 9750 3200 50  0001 C CNN
@@
 $EndComp
 $Comp
-L +5V #PWR4
+L +5V #PWR019
 U 1 1 59068316
 P 9600 1150
-F 0 "#PWR4" H 9600 1000 50  0001 C CNN
+F 0 "#PWR019" H 9600 1000 50  0001 C CNN
 F 1 "+5V" H 9550 1350 50  0000 C CNN
 F 2 "" H 9600 1150 50  0001 C CNN
@@
 $EndComp
 $Comp
-L GND #PWR13
+L GND #PWR020
 U 1 1 5906D186
 P 1400 5000
-F 0 "#PWR13" H 1400 4750 50  0001 C CNN
+F 0 "#PWR020" H 1400 4750 50  0001 C CNN
 F 1 "GND" H 1405 4827 50  0000 C CNN
 F 2 "" H 1400 5000 50  0001 C CNN
@@
 $EndComp
 $Comp
-L GND #PWR14
+L GND #PWR021
 U 1 1 5906DA5E
 P 1800 5000
-F 0 "#PWR14" H 1800 4750 50  0001 C CNN
+F 0 "#PWR021" H 1800 4750 50  0001 C CNN
 F 1 "GND" H 1805 4827 50  0000 C CNN
 F 2 "" H 1800 5000 50  0001 C CNN
@@
 $EndComp
 $Comp
-L +3V3 #PWR9
+L +3V3 #PWR022
 U 1 1 590700EE
 P 1800 3800
-F 0 "#PWR9" H 1800 3650 50  0001 C CNN
+F 0 "#PWR022" H 1800 3650 50  0001 C CNN
 F 1 "+3V3" H 1815 3973 50  0000 C CNN
 F 2 "" H 1800 3800 50  0001 C CNN
@@
 	1800 3800 1800 3900
 $Comp
-L GND #PWR6
+L GND #PWR023
 U 1 1 590717B1
 P 3150 2300
-F 0 "#PWR6" H 3150 2050 50  0001 C CNN
+F 0 "#PWR023" H 3150 2050 50  0001 C CNN
 F 1 "GND" H 3155 2127 50  0000 C CNN
 F 2 "" H 3150 2300 50  0001 C CNN
@@
 	2000 1900 1750 1900
 $Comp
-L GND #PWR7
+L GND #PWR024
 U 1 1 5907D79F
 P 1900 3050
-F 0 "#PWR7" H 1900 2800 50  0001 C CNN
+F 0 "#PWR024" H 1900 2800 50  0001 C CNN
 F 1 "GND" H 1905 2877 50  0000 C CNN
 F 2 "" H 1900 3050 50  0001 C CNN
@@
 $EndComp
 $Comp
-L +3V3 #PWR2
+L +3V3 #PWR025
 U 1 1 59083691
 P 8300 850
-F 0 "#PWR2" H 8300 700 50  0001 C CNN
+F 0 "#PWR025" H 8300 700 50  0001 C CNN
 F 1 "+3V3" H 8315 1023 50  0000 C CNN
 F 2 "" H 8300 850 50  0001 C CNN
@@
 $EndComp
 $Comp
-L GND #PWR12
+L GND #PWR026
 U 1 1 59083A6B
 P 8300 3850
-F 0 "#PWR12" H 8300 3600 50  0001 C CNN
+F 0 "#PWR026" H 8300 3600 50  0001 C CNN
 F 1 "GND" H 8305 3677 50  0000 C CNN
 F 2 "" H 8300 3850 50  0001 C CNN

Commit message: added mounting holes
added a lot of capacitors (there was some room left ;) )

layout nearly finished
logos are missing ;)
not much work left I think
Parts:
- added M1, M2: mounting hole, Mounting_Holes:MountingHole_3.2mm_M3_Pad_Via, symbol Screw_Terminal_1x01
Connections:
- net GND: now also M1.1, M2.1
Changed lines of the file:
@@
 	3300 2700 3350 2700
 Connection ~ 3300 2900
+$Comp
+L Screw_Terminal_1x01 M1
+U 1 1 59079FB2
+P 10450 4100
+F 0 "M1" H 10370 4054 50  0000 R CNN
+F 1 "mounting hole" H 10370 4145 50  0000 R CNN
+F 2 "Mounting_Holes:MountingHole_3.2mm_M3_Pad_Via" H 10450 3975 50  0001 C CNN
+F 3 "" H 10450 4000 50  0001 C CNN
+	1    10450 4100
+	-1   0    0    1
+$EndComp
+$Comp
+L Screw_Terminal_1x01 M2
+U 1 1 5907B01E
+P 10450 4300
+F 0 "M2" H 10370 4254 50  0000 R CNN
+F 1 "mounting hole" H 10370 4345 50  0000 R CNN
+F 2 "Mounting_Holes:MountingHole_3.2mm_M3_Pad_Via" H 10450 4175 50  0001 C CNN
+F 3 "" H 10450 4200 50  0001 C CNN
+	1    10450 4300
+	-1   0    0    1
+$EndComp
+$Comp
+L GND #PWR?
+U 1 1 5907B64D
+P 10200 4400
+F 0 "#PWR?" H 10200 4150 50  0001 C CNN
+F 1 "GND" H 10205 4227 50  0000 C CNN
+F 2 "" H 10200 4400 50  0000 C CNN
+F 3 "" H 10200 4400 50  0000 C CNN
+	1    10200 4400
+	1    0    0    -1
+$EndComp
+Wire Wire Line
+	10200 4400 10200 4100
+Wire Wire Line
+	10200 4100 10250 4100
+Wire Wire Line
+	10250 4300 10200 4300
+Connection ~ 10200 4300
 $EndSCHEMATC
